File: Alius_6502.kicad_sch (KiCad schematic)
At the start: 28 parts, among them J1 Conn_01x02_Male, J2 Conn_01x20, J3 Power, J4 SD_Card, SW1 SW_Push, U1 WDC65C02, U2 74HC00, U3 74HC02, U4 28C256, U5 74HC21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

Commit message: Version 1.2
Improved reset.
Added connection for PWM display brightness.

NOTE: This board revision is yet to be made and tested.
Parts:
- C1: footprint Capacitor_THT:CP_Radial_D6.3mm_P2.50mm -> Alius_6502:CP_Radial_D6.3mm_P2.50mm
- C2, C3, C4, C5, C6, C7, C8, C9: footprint Capacitor_THT:C_Axial_L3.8mm_D2.6mm_P7.50mm_Horizontal -> Alius_6502:C_Axial_L3.8mm_D2.6mm_P7.50mm_Horizontal
- J1, J3: symbol Connector:Conn_01x02_Male -> Connector:Conn_01x02_Pin
- J4: symbol Connector:Conn_01x08_Male -> Connector:Conn_01x08_Pin
- U1, U7, U8: footprint Alius_6502:40_PIN_PDIP -> Alius_6502:40-pin-DIP
- U2, U3, U5: footprint Package_DIP:DIP-14_W7.62mm_Socket_LongPads -> Alius_6502:DIP-14_W7.62mm_Socket_LongPads
- U4: footprint Package_DIP:DIP-28_W15.24mm_LongPads -> Alius_6502:28-pin-DIP
- U6: footprint Package_DIP:DIP-28_W15.24mm_LongPads -> Alius_6502:28-pin-DIP; symbol Alius:62256 -> Alius:RAM62256
Connections:
- net RESET: now also U3.13 (4Y); no longer C1.1, R3.2, SW1.2
- net DisplayPWM: now reaches U8.19 (CB2)
- net at U3.10 (3Y): now also U3.11 (4A), U3.12 (4B)
- net +5V renamed VCC
- net VCC: no longer U3.11 (4A), U3.12 (4B), U3.8 (3A), U3.9 (3B)
- new net RESET_BTN: C1.1, R3.2, SW1.2, U3.8 (3A), U3.9 (3B)
- no-connect marks 24 -> 21
